Commit message: Created a gazebo launch file for the mobile robot

File: my_robot_description/urdf/common_properties.xacro (robot description, xacro)
@@ -7,3 +7,30 @@
         <color rgba="0.5 0.5 0.5 1"/>
     </material>
+    <xacro:macro name="box_inertia" params="m l w h xyz rpy">
+        <inertial>
+            <origin xyz="${xyz}" rpy="${rpy}"/>
+            <mass value="${m}"/>
+            <inertia ixx="${(1/12)*m*(h*h + l*l)}" ixy="0" ixz="0"
+                     iyy="${(1/12)*m*(w*w + l*l)}" iyz="0"
+                     izz="${(1/12)*m*(w*w + h*h)}"/>
+        </inertial>
+    </xacro:macro>
+    <xacro:macro name="cylinder_inertia" params="m r h xyz rpy">
+        <inertial>
+            <origin xyz="${xyz}" rpy="${rpy}"/>
+            <mass value="${m}"/>
+            <inertia ixx="${(1/12)*m*(3*r*r + h*h)}" ixy="0" ixz="0"
+                     iyy="${(1/12)*m*(3*r*r + h*h)}" iyz="0"
+                     izz="${(1/2)*m*r*r}"/>
+        </inertial>
+    </xacro:macro>
+    <xacro:macro name="sphere_inertia" params="m r xyz rpy">
+        <inertial>
+            <origin xyz="${xyz}" rpy="${rpy}"/>
+            <mass value="${m}"/>
+            <inertia ixx="${(2/5)*m*r*r}" ixy="0" ixz="0"
+                     iyy="${(2/5)*m*r*r}" iyz="0"
+                     izz="${(2/5)*m*r*r}"/>
+        </inertial>
+    </xacro:macro>
 </robot>

File: my_robot_description/urdf/mobile_base.xacro (robot description, xacro)
@@ -15,4 +15,12 @@
                 <material name="grey"/>
             </visual>
+            <collision>
+                <geometry>
+                    <cylinder radius="${wheel_radius}" length="${wheel_length}"/>
+                </geometry>
+                <origin xyz="0 0 0" rpy="${pi/2} 0 0"/>
+            </collision>
+            <xacro:cylinder_inertia m="1" r="${wheel_radius}" h="${wheel_length}"
+                                    xyz="0 0 0" rpy="${pi/2} 0 0"/>
         </link>
     </xacro:macro>
@@ -28,5 +36,13 @@
             <material name="teal" />
         </visual>
-    </link>g m
+        <collision>
+            <geometry>
+                <box size="${base_length} ${base_width} ${base_height}" />
+            </geometry>
+            <origin xyz="0 0 ${base_height/2} " rpy="0 0 0" />
+        </collision>
+        <xacro:box_inertia m="5" l="${base_length}" w="${base_width}" h="${base_height}"
+                            xyz="0 0 ${base_height/2}" rpy="0 0 0"/>
+    </link>
     <link name="caster_wheel_link">
         <visual>
@@ -37,4 +53,11 @@
             <material name="grey"/>
         </visual>
+        <collision>
+            <geometry>
+                <sphere radius="${wheel_radius/2}"/>
+            </geometry>
+            <origin xyz="0 0 0" rpy="0 0 0"/>
+        </collision>
+        <xacro:sphere_inertia m="0.5" r="${wheel_radius/2}" xyz="0 0 0" rpy="0 0 0"/>
     </link>
     <joint name="base_footprint_base_joint" type="fixed">
