Commit message: save before trying to get gz garden plugins workin

File: my_robot_description/urdf/mobile_base.xacro (robot description, xacro)
@@ -1,8 +1,8 @@
 <?xml version="1.0"?>
 <robot xmlns:xacro="http://www.ros.org/wiki/xacro">
-    <xacro:property name="base_length" value="0.8"/>
-    <xacro:property name="base_width" value="0.6"/>
-    <xacro:property name="base_height" value="0.3"/>
-    <xacro:property name="wheel_radius" value="0.2"/>
+    <xacro:property name="base_length" value="0.6"/>
+    <xacro:property name="base_width" value="0.4"/>
+    <xacro:property name="base_height" value="0.2"/>
+    <xacro:property name="wheel_radius" value="0.1"/>
     <xacro:property name="wheel_length" value="0.05"/>
     <xacro:macro name="wheel_link" params="prefix">
@@ -21,5 +21,5 @@
                 <origin xyz="0 0 0" rpy="${pi/2} 0 0"/>
             </collision>
-            <xacro:cylinder_inertia m="1" r="${wheel_radius}" h="${wheel_length}"
+            <xacro:cylinder_inertia m="1" r="${2*wheel_radius}" h="${2*wheel_length}"
                                     xyz="0 0 0" rpy="${pi/2} 0 0"/>
         </link>
@@ -42,5 +42,5 @@
             <origin xyz="0 0 ${base_height/2} " rpy="0 0 0" />
         </collision>
-        <xacro:box_inertia m="5" l="${base_length}" w="${base_width}" h="${base_height}"
+        <xacro:box_inertia m="5" l="${2*base_length}" w="${2*base_width}" h="${2*base_height}"
                             xyz="0 0 ${base_height/2}" rpy="0 0 0"/>
     </link>
@@ -59,5 +59,5 @@
             <origin xyz="0 0 0" rpy="0 0 0"/>
         </collision>
-        <xacro:sphere_inertia m="0.5" r="${wheel_radius/2}" xyz="0 0 0" rpy="0 0 0"/>
+        <xacro:sphere_inertia m="0.5" r="${2*wheel_radius/2}" xyz="0 0 0" rpy="0 0 0"/>
     </link>
     <joint name="base_footprint_base_joint" type="fixed">

File: my_robot_description/urdf/my_robot.urdf.xacro (robot description, xacro)
@@ -3,3 +3,5 @@
     <xacro:include filename="common_properties.xacro"/>
     <xacro:include filename="mobile_base.xacro"/>
+    <xacro:include filename="mobile_base_gazebo.xacro"/>
+    <xacro:include filename="camera.xacro"/>
 </robot>
