Commit message: Install yolo and got image detection working

File: my_robot_description/urdf/camera.xacro (robot description, xacro)
@@ -1,26 +1,27 @@
 <?xml version="1.0"?>
 <robot xmlns:xacro="http://www.ros.org/wiki/xacro">
-    <xacro:property name="camera_length" value="0.01"/>
-    <xacro:property name="camera_width" value="0.1"/>
-    <xacro:property name="camera_height" value="0.05"/>
+    <xacro:property name="camera_length" value="0.01" />
+    <xacro:property name="camera_width" value="0.1" />
+    <xacro:property name="camera_height" value="0.05" />
     <link name="camera_link">
         <visual>
             <geometry>
-                <box size="${camera_length} ${camera_width} ${camera_height}"/>
+                <box size="${camera_length} ${camera_width} ${camera_height}" />
             </geometry>
-            <material name="grey"/>
+            <material name="grey" />
         </visual>
         <collision>
             <geometry>
-                <box size="${camera_length} ${camera_width} ${camera_height}"/>
+                <box size="${camera_length} ${camera_width} ${camera_height}" />
             </geometry>
-            <material name="grey"/>
+            <material name="grey" />
         </collision>
-        <xacro:box_inertia m="0.1" l="${camera_length}" w="${camera_width}" h="${camera_height}" xyz="0 0 0" rpy="0 0 0"/>
+        <xacro:box_inertia m="0.1" l="${camera_length}" w="${camera_width}" h="${camera_height}"
+            xyz="0 0 0" rpy="0 0 0" />
     </link>
     <joint name="base_camera_joint" type="fixed">
-        <parent link="base_link"/>
-        <child link="camera_link"/>
-        <origin xyz="${(base_length + camera_length)/2} 0 ${base_height/2}" rpy="0 0 0"/>
+        <parent link="base_link" />
+        <child link="camera_link" />
+        <origin xyz="${(base_length + camera_length)/2} 0 ${base_height/2}" rpy="0 0 0" />
     </joint>
     <gazebo reference="camera_link">

File: my_robot_description/urdf/common_properties.xacro (robot description, xacro)
@@ -5,31 +5,39 @@
     </material>
     <material name="grey">
-        <color rgba="0.5 0.5 0.5 1"/>
+        <color rgba="0.5 0.5 0.5 1" />
+    </material>
+    <!-- material orange -->
+    <material name="orange">
+        <color rgba="1 0.5 0 1" />
+    </material>
+    <!-- material yellow -->
+    <material name="yellow">
+        <color rgba="1 1 0 1" />
     </material>
     <xacro:macro name="box_inertia" params="m l w h xyz rpy">
         <inertial>
-            <origin xyz="${xyz}" rpy="${rpy}"/>
-            <mass value="${m}"/>
+            <origin xyz="${xyz}" rpy="${rpy}" />
+            <mass value="${m}" />
             <inertia ixx="${(1/12)*m*(h*h + l*l)}" ixy="0" ixz="0"
-                     iyy="${(1/12)*m*(w*w + l*l)}" iyz="0"
-                     izz="${(1/12)*m*(w*w + h*h)}"/>
+                iyy="${(1/12)*m*(w*w + l*l)}" iyz="0"
+                izz="${(1/12)*m*(w*w + h*h)}" />
         </inertial>
     </xacro:macro>
     <xacro:macro name="cylinder_inertia" params="m r h xyz rpy">
         <inertial>
-            <origin xyz="${xyz}" rpy="${rpy}"/>
-            <mass value="${m}"/>
+            <origin xyz="${xyz}" rpy="${rpy}" />
+            <mass value="${m}" />
             <inertia ixx="${(1/12)*m*(3*r*r + h*h)}" ixy="0" ixz="0"
-                     iyy="${(1/12)*m*(3*r*r + h*h)}" iyz="0"
-                     izz="${(1/2)*m*r*r}"/>
+                iyy="${(1/12)*m*(3*r*r + h*h)}" iyz="0"
+                izz="${(1/2)*m*r*r}" />
         </inertial>
     </xacro:macro>
     <xacro:macro name="sphere_inertia" params="m r xyz rpy">
         <inertial>
-            <origin xyz="${xyz}" rpy="${rpy}"/>
-            <mass value="${m}"/>
+            <origin xyz="${xyz}" rpy="${rpy}" />
+            <mass value="${m}" />
             <inertia ixx="${(2/5)*m*r*r}" ixy="0" ixz="0"
-                     iyy="${(2/5)*m*r*r}" iyz="0"
-                     izz="${(2/5)*m*r*r}"/>
+                iyy="${(2/5)*m*r*r}" iyz="0"
+                izz="${(2/5)*m*r*r}" />
         </inertial>
     </xacro:macro>

File: my_robot_description/urdf/mobile_base.xacro (robot description, xacro)
@@ -1,31 +1,31 @@
 <?xml version="1.0"?>
 <robot xmlns:xacro="http://www.ros.org/wiki/xacro">
-    <xacro:property name="base_length" value="0.6"/>
-    <xacro:property name="base_width" value="0.4"/>
-    <xacro:property name="base_height" value="0.2"/>
-    <xacro:property name="wheel_radius" value="0.1"/>
-    <xacro:property name="wheel_length" value="0.05"/>
+    <xacro:property name="base_length" value="0.6" />
+    <xacro:property name="base_width" value="0.4" />
+    <xacro:property name="base_height" value="0.2" />
+    <xacro:property name="wheel_radius" value="0.1" />
+    <xacro:property name="wheel_length" value="0.05" />
     <xacro:macro name="wheel_link" params="prefix">
         <link name="${prefix}_wheel_link">
             <visual>
                 <geometry>
-                    <cylinder radius="${wheel_radius}" length="${wheel_length}"/>
+                    <cylinder radius="${wheel_radius}" length="${wheel_length}" />
                 </geometry>
-                <origin xyz="0 0 0" rpy="${pi/2} 0 0"/>
-                <material name="grey"/>
+                <origin xyz="0 0 0" rpy="${pi/2} 0 0" />
+                <material name="grey" />
             </visual>
             <collision>
                 <geometry>
-                    <cylinder radius="${wheel_radius}" length="${wheel_length}"/>
+                    <cylinder radius="${wheel_radius}" length="${wheel_length}" />
                 </geometry>
-                <origin xyz="0 0 0" rpy="${pi/2} 0 0"/>
+                <origin xyz="0 0 0" rpy="${pi/2} 0 0" />
             </collision>
             <xacro:cylinder_inertia m="1" r="${2*wheel_radius}" h="${2*wheel_length}"
-                                    xyz="0 0 0" rpy="${pi/2} 0 0"/>
+                xyz="0 0 0" rpy="${pi/2} 0 0" />
         </link>
     </xacro:macro>
-    <xacro:wheel_link prefix="right"/>
-    <xacro:wheel_link prefix="left"/>
-    <link name="base_footprint_link"/>
+    <xacro:wheel_link prefix="right" />
+    <xacro:wheel_link prefix="left" />
+    <link name="base_footprint_link" />
     <link name="base_link">
         <visual>
@@ -43,43 +43,43 @@
         </collision>
         <xacro:box_inertia m="5" l="${2*base_length}" w="${2*base_width}" h="${2*base_height}"
-                            xyz="0 0 ${base_height/2}" rpy="0 0 0"/>
+            xyz="0 0 ${base_height/2}" rpy="0 0 0" />
     </link>
     <link name="caster_wheel_link">
         <visual>
             <geometry>
-                <sphere radius="${wheel_radius/2}"/>
+                <sphere radius="${wheel_radius/2}" />
             </geometry>
-            <origin xyz="0 0 0" rpy="0 0 0"/>
-            <material name="grey"/>
+            <origin xyz="0 0 0" rpy="0 0 0" />
+            <material name="grey" />
         </visual>
         <collision>
             <geometry>
-                <sphere radius="${wheel_radius/2}"/>
+                <sphere radius="${wheel_radius/2}" />
             </geometry>
-            <origin xyz="0 0 0" rpy="0 0 0"/>
+            <origin xyz="0 0 0" rpy="0 0 0" />
         </collision>
-        <xacro:sphere_inertia m="0.5" r="${2*wheel_radius/2}" xyz="0 0 0" rpy="0 0 0"/>
+        <xacro:sphere_inertia m="0.5" r="${2*wheel_radius/2}" xyz="0 0 0" rpy="0 0 0" />
     </link>
     <joint name="base_footprint_base_joint" type="fixed">
-        <parent link="base_footprint_link"/>
-        <child link="base_link"/>
-        <origin xyz="0 0 ${wheel_radius}" rpy="0 0 0"/>
+        <parent link="base_footprint_link" />
+        <child link="base_link" />
+        <origin xyz="0 0 ${wheel_radius}" rpy="0 0 0" />
     </joint>
     <joint name="base_right_wheel_joint" type="continuous">
-        <parent link="base_link"/>
-        <child link="right_wheel_link"/>
-        <origin xyz="${-base_length/4} ${-base_width/2 - wheel_length/2} 0" rpy="0 0 0"/>
-        <axis xyz="0 1 0"/>
+        <parent link="base_link" />
+        <child link="right_wheel_link" />
+        <origin xyz="${-base_length/4} ${-base_width/2 - wheel_length/2} 0" rpy="0 0 0" />
+        <axis xyz="0 1 0" />
     </joint>
     <joint name="base_left_wheel_joint" type="continuous">
-        <parent link="base_link"/>
-        <child link="left_wheel_link"/>
-        <origin xyz="${-base_length/4} ${base_width/2 + wheel_length/2} 0" rpy="0 0 0"/>
-        <axis xyz="0 1 0"/>
+        <parent link="base_link" />
+        <child link="left_wheel_link" />
+        <origin xyz="${-base_length/4} ${base_width/2 + wheel_length/2} 0" rpy="0 0 0" />
+        <axis xyz="0 1 0" />
     </joint>
     <joint name="base_caster_wheel_joint" type="fixed">
-        <parent link="base_link"/>
-        <child link="caster_wheel_link"/>
-        <origin xyz="${base_length/3} 0 ${-wheel_radius/2}" rpy="0 0 0"/>
+        <parent link="base_link" />
+        <child link="caster_wheel_link" />
+        <origin xyz="${base_length/3} 0 ${-wheel_radius/2}" rpy="0 0 0" />
     </joint>
 </robot>

File: my_robot_description/urdf/mobile_base_gazebo.xacro (robot description, xacro)
@@ -12,6 +12,6 @@
     <gazebo reference="caster_wheel_link">
         <material>Gazebo/Orange</material>
-        <mu1 value="0.1"/>
-        <mu2 value="0.2"/>
+        <mu1 value="0.1" />
+        <mu2 value="0.2" />
     </gazebo>
     <gazebo>

File: my_robot_description/urdf/my_robot.urdf.xacro (robot description, xacro)
@@ -1,7 +1,15 @@
 <?xml version="1.0"?>
 <robot name="my_robot" xmlns:xacro="http://www.ros.org/wiki/xacro">
-    <xacro:include filename="common_properties.xacro"/>
-    <xacro:include filename="mobile_base.xacro"/>
-    <xacro:include filename="mobile_base_gazebo.xacro"/>
-    <xacro:include filename="camera.xacro"/>
+    <xacro:include filename="common_properties.xacro" />
+    <xacro:include filename="mobile_base.xacro" />
+    <xacro:include filename="mobile_base_gazebo.xacro" />
+    <xacro:include filename="camera.xacro" />
+      <!-- create a joint called  base_arm_base_joint with the origin of the arm_base_link rotate 90
+    degrees on the y-axis and transformed 0.3 in the x direction and 0.1 up -->
+    <joint name="mobile_base_arm_joint" type="fixed">
+        <origin xyz="${0.25*base_length} 0 ${base_height}" rpy="0 0 0" />
+        <parent link="base_link" />
+        <child link="arm_base_link" />
+    </joint>
+    <xacro:include filename="arm.xacro" />
 </robot>
