Commit message: create launch folder for arduinobot with rviz

File: arduinobot_description/urdf/arduinobot.urdf.xacro (robot description, xacro)
@@ -1,9 +1,13 @@
-<!-- standard urdf xacro file -->
-<? xml version="1.0"?>
+<?xml version="1.0"?>
 <robot xmlns:xacro="http://www.ros.org/wiki/xacro" name="arduinobot">
+    <!-- variables -->
+    <xacro:property name="PI" value="3.14159265359" />
+    <xacro:property name="velocity" value="10.0" />
+    <xacro:property name="effort" value="30.0" />
+    <!-- links -->
     <link name="world" />
     <link name="base_link">
         <visual>
-            <origin xyz="0 0 0" rpy="0 0 0" />
+            <origin xyz="-0.5 -0.5 0" rpy="0 0 0" />
             <geometry>
                 <mesh filename="package://arduinobot_description/meshes/basement.STL"
@@ -11,5 +15,67 @@
             </geometry>
         </visual>
+        <collision>
+            <origin xyz="-0.5 -0.5 0" rpy="0 0 0" />
+            <geometry>
+                <mesh filename="package://arduinobot_description/meshes/basement.STL"
+                    scale="0.01 0.01 0.01" />
+            </geometry>
+        </collision>
     </link>
+    <link name="base_plate_link">
+        <visual>
+            <origin xyz="-0.39 -0.39 -0.56" rpy="0 0 0" />
+            <geometry>
+                <mesh filename="package://arduinobot_description/meshes/base_plate.STL"
+                    scale="0.01 0.01 0.01" />
+            </geometry>
+        </visual>
+    </link>
+    <link name="forward_drive_arm_link">
+        <visual>
+            <origin xyz="0.19 0.06 -0.08" rpy="0 -${PI/2} ${PI/2}" />
+            <geometry>
+                <mesh filename="package://arduinobot_description/meshes/forward_drive_arm.STL"
+                    scale="0.01 0.01 0.01" />
+            </geometry>
+        </visual>
+    </link>
+    <link name="horizontal_arm_link">
+        <visual>
+            <origin xyz="-0.03 -0.4 -0.06" rpy="${PI/2} 0 ${PI/2}" />
+            <geometry>
+                <mesh filename="package://arduinobot_description/meshes/horizontal_arm.STL"
+                    scale="0.01 0.01 0.01" />
+            </geometry>
+        </visual>
+    </link>
+    <link name="claw_support_link">
+        <visual>
+            <origin xyz="0 -0.05 -0.15" rpy="0 0 ${PI/2}" />
+            <geometry>
+                <mesh filename="package://arduinobot_description/meshes/claw_support.STL"
+                    scale="0.01 0.01 0.01" />
+            </geometry>
+        </visual>
+    </link>
+    <link name="gripper_right_link">
+        <visual>
+            <origin xyz="-0.1 0.5 -0.1" rpy="0 0 -${PI/2}" />
+            <geometry>
+                <mesh filename="package://arduinobot_description/meshes/right_finger.STL"
+                    scale="0.01 0.01 0.01" />
+            </geometry>
+        </visual>
+    </link>
+    <link name="gripper_left_link">
+        <visual>
+            <origin xyz="-0.04 0.5 -0.1" rpy="0 0 -${PI/2}" />
+            <geometry>
+                <mesh filename="package://arduinobot_description/meshes/left_finger.STL"
+                    scale="0.01 0.01 0.01" />
+            </geometry>
+        </visual>
+    </link>
+    <!-- joints -->
     <joint name="virtual_joint" type="fixed">
         <parent link="world" />
@@ -17,3 +83,44 @@
         <origin xyz="0 0 0" rpy="0 0 0" />
     </joint>
+    <joint name="base_base_plate_joint_1" type="revolute">
+        <parent link="base_link" />
+        <child link="base_plate_link" />
+        <origin xyz="0 0 0.307" rpy="0 0 0" />
+        <axis xyz="0 0 1" />
+        <limit lower="-${PI/2}" upper="${PI/2}" effort="${effort}" velocity="${velocity}" />
+    </joint>
+    <joint name="base_plate_forward_drive_arm_joint_2" type="revolute">
+        <parent link="base_plate_link" />
+        <child link="forward_drive_arm_link" />
+        <origin xyz="-0.02 0 0.35" rpy="0 0 0" />
+        <axis xyz="1 0 0" />
+        <limit lower="-${PI/2}" upper="${PI/2}" effort="${effort}" velocity="${velocity}" />
+    </joint>
+    <joint name="forward_drive_arm_horizontal_arm_joint_3" type="revolute">
+        <parent link="forward_drive_arm_link" />
+        <child link="horizontal_arm_link" />
+        <origin xyz="0 0 0.8" rpy="0 0 0" />
+        <axis xyz="1 0 0" />
+        <limit lower="-${PI/2}" upper="${PI/2}" effort="${effort}" velocity="${velocity}" />
+    </joint>
+    <joint name="horizontal_arm_claw_support_joint" type="fixed">
+        <parent link="horizontal_arm_link" />
+        <child link="claw_support_link" />
+        <origin xyz="0 0.82 0" rpy="0 0 0" />
+    </joint>
+    <joint name="claw_support_gripper_right_joint_4" type="revolute">
+        <parent link="claw_support_link" />
+        <child link="gripper_right_link" />
+        <origin xyz="-0.04 0.13 -0.1" rpy="0 0 0" />
+        <axis xyz="0 0 1" />
+        <limit lower="-${PI/2}" upper="0.0" effort="${effort}" velocity="${velocity}" />
+    </joint>
+    <joint name="claw_support_gripper_left_joint_5" type="revolute">
+        <parent link="claw_support_link" />
+        <child link="gripper_left_link" />
+        <origin xyz="-0.22 0.13 -0.1" rpy="0 0 0" />
+        <axis xyz="0 0 1" />
+        <limit lower="0.0" upper="${PI/2}" effort="${effort}" velocity="${velocity}" />
+        <mimic joint="claw_support_gripper_right_joint_4" multiplier="-1" offset="0" />
+    </joint>
 </robot>

Commit message: add support for gazebo

File: arduinobot_description/urdf/arduinobot.urdf.xacro (robot description, xacro)
@@ -5,7 +5,16 @@
     <xacro:property name="velocity" value="10.0" />
     <xacro:property name="effort" value="30.0" />
+    <xacro:macro name="default_inertial" params="mass">
+        <inertial>
+            <mass value="${mass}" />
+            <inertia ixx="1.0" ixy="0.0" ixz="0.0"
+                iyy="1.0" iyz="0.0"
+                izz="1.0" />
+        </inertial>
+    </xacro:macro>
     <!-- links -->
     <link name="world" />
     <link name="base_link">
+        <xacro:default_intertial mass="1.0" />
         <visual>
             <origin xyz="-0.5 -0.5 0" rpy="0 0 0" />
@@ -24,4 +33,5 @@
     </link>
     <link name="base_plate_link">
+        <xacro:default_intertial mass="0.1" />
         <visual>
             <origin xyz="-0.39 -0.39 -0.56" rpy="0 0 0" />
@@ -31,6 +41,14 @@
             </geometry>
         </visual>
+        <collision>
+            <origin xyz="-0.39 -0.39 -0.56" rpy="0 0 0" />
+            <geometry>
+                <mesh filename="package://arduinobot_description/meshes/base_plate.STL"
+                    scale="0.01 0.01 0.01" />
+            </geometry>
+        </collision>
     </link>
     <link name="forward_drive_arm_link">
+        <xacro:default_intertial mass="0.1" />
         <visual>
             <origin xyz="0.19 0.06 -0.08" rpy="0 -${PI/2} ${PI/2}" />
@@ -40,6 +58,14 @@
             </geometry>
         </visual>
+        <collision>
+            <origin xyz="0.19 0.06 -0.08" rpy="0 -${PI/2} ${PI/2}" />
+            <geometry>
+                <mesh filename="package://arduinobot_description/meshes/forward_drive_arm.STL"
+                    scale="0.01 0.01 0.01" />
+            </geometry>
+        </collision>
     </link>
     <link name="horizontal_arm_link">
+        <xacro:default_intertial mass="0.1" />
         <visual>
             <origin xyz="-0.03 -0.4 -0.06" rpy="${PI/2} 0 ${PI/2}" />
@@ -49,6 +75,14 @@
             </geometry>
         </visual>
+        <collision>
+            <origin xyz="-0.03 -0.4 -0.06" rpy="${PI/2} 0 ${PI/2}" />
+            <geometry>
+                <mesh filename="package://arduinobot_description/meshes/horizontal_arm.STL"
+                    scale="0.01 0.01 0.01" />
+            </geometry>
+        </collision>
     </link>
     <link name="claw_support_link">
+        <xacro:default_intertial mass="0.05" />
         <visual>
             <origin xyz="0 -0.05 -0.15" rpy="0 0 ${PI/2}" />
@@ -58,6 +92,14 @@
             </geometry>
         </visual>
+        <collision>
+            <origin xyz="0 -0.05 -0.15" rpy="0 0 ${PI/2}" />
+            <geometry>
+                <mesh filename="package://arduinobot_description/meshes/claw_support.STL"
+                    scale="0.01 0.01 0.01" />
+            </geometry>
+        </collision>
     </link>
     <link name="gripper_right_link">
+        <xacro:default_intertial mass="0.01" />
         <visual>
             <origin xyz="-0.1 0.5 -0.1" rpy="0 0 -${PI/2}" />
@@ -67,6 +109,14 @@
             </geometry>
         </visual>
+        <collision>
+            <origin xyz="-0.1 0.5 -0.1" rpy="0 0 -${PI/2}" />
+            <geometry>
+                <mesh filename="package://arduinobot_description/meshes/right_finger.STL"
+                    scale="0.01 0.01 0.01" />
+            </geometry>
+        </collision>
     </link>
     <link name="gripper_left_link">
+        <xacro:default_intertial mass="0.01" />
         <visual>
             <origin xyz="-0.04 0.5 -0.1" rpy="0 0 -${PI/2}" />
@@ -76,4 +126,11 @@
             </geometry>
         </visual>
+        <collision>
+            <origin xyz="-0.04 0.5 -0.1" rpy="0 0 -${PI/2}" />
+            <geometry>
+                <mesh filename="package://arduinobot_description/meshes/left_finger.STL"
+                    scale="0.01 0.01 0.01" />
+            </geometry>
+        </collision>
     </link>
     <!-- joints -->

Commit message: Create gazebo and ros2_control xacro

File: arduinobot_description/urdf/arduinobot.urdf.xacro (robot description, xacro)
@@ -1,8 +1,12 @@
 <?xml version="1.0"?>
 <robot xmlns:xacro="http://www.ros.org/wiki/xacro" name="arduinobot">
+    <!-- includes -->
+    <xacro:include filename="$(find arduinobot_description)/urdf/arduinobot_gazebo_xacro" />
+    <xacro:include filename="$(find arduinobot_description)/urdf/arduinobot_ros2_control.xacro" />
     <!-- variables -->
     <xacro:property name="PI" value="3.14159265359" />
     <xacro:property name="velocity" value="10.0" />
     <xacro:property name="effort" value="30.0" />
+    <!-- macros -->
     <xacro:macro name="default_inertial" params="mass">
         <inertial>
@@ -13,8 +17,17 @@
         </inertial>
     </xacro:macro>
+    <xacro:macro name="default_transmission" params="number">
+        <transmission name="transmission_${number}">
+            <plugin>transmission_interface/SimpleTransmission</plugin>
+            <actuator name="motor_${number}" role="actuator1"/>
+            <joint name="joint_${number}" role="joint1">
+                <mechanical_reducation>1.0</mechanical_reducation>
+            </joint>
+        </transmission>
+    </xacro:macro>
     <!-- links -->
     <link name="world" />
     <link name="base_link">
-        <xacro:default_intertial mass="1.0" />
+        <xacro:default_inertial mass="1.0" />
         <visual>
             <origin xyz="-0.5 -0.5 0" rpy="0 0 0" />
@@ -33,5 +46,5 @@
     </link>
     <link name="base_plate_link">
-        <xacro:default_intertial mass="0.1" />
+        <xacro:default_inertial mass="0.1" />
         <visual>
             <origin xyz="-0.39 -0.39 -0.56" rpy="0 0 0" />
@@ -50,5 +63,5 @@
     </link>
     <link name="forward_drive_arm_link">
-        <xacro:default_intertial mass="0.1" />
+        <xacro:default_inertial mass="0.1" />
         <visual>
             <origin xyz="0.19 0.06 -0.08" rpy="0 -${PI/2} ${PI/2}" />
@@ -67,5 +80,5 @@
     </link>
     <link name="horizontal_arm_link">
-        <xacro:default_intertial mass="0.1" />
+        <xacro:default_inertial mass="0.1" />
         <visual>
             <origin xyz="-0.03 -0.4 -0.06" rpy="${PI/2} 0 ${PI/2}" />
@@ -84,5 +97,5 @@
     </link>
     <link name="claw_support_link">
-        <xacro:default_intertial mass="0.05" />
+        <xacro:default_inertial mass="0.05" />
         <visual>
             <origin xyz="0 -0.05 -0.15" rpy="0 0 ${PI/2}" />
@@ -101,5 +114,5 @@
     </link>
     <link name="gripper_right_link">
-        <xacro:default_intertial mass="0.01" />
+        <xacro:default_inertial mass="0.01" />
         <visual>
             <origin xyz="-0.1 0.5 -0.1" rpy="0 0 -${PI/2}" />
@@ -118,5 +131,5 @@
     </link>
     <link name="gripper_left_link">
-        <xacro:default_intertial mass="0.01" />
+        <xacro:default_inertial mass="0.01" />
         <visual>
             <origin xyz="-0.04 0.5 -0.1" rpy="0 0 -${PI/2}" />
@@ -140,5 +153,5 @@
         <origin xyz="0 0 0" rpy="0 0 0" />
     </joint>
-    <joint name="base_base_plate_joint_1" type="revolute">
+    <joint name="joint_1" type="revolute">
         <parent link="base_link" />
         <child link="base_plate_link" />
@@ -147,5 +160,5 @@
         <limit lower="-${PI/2}" upper="${PI/2}" effort="${effort}" velocity="${velocity}" />
     </joint>
-    <joint name="base_plate_forward_drive_arm_joint_2" type="revolute">
+    <joint name="joint_2" type="revolute">
         <parent link="base_plate_link" />
         <child link="forward_drive_arm_link" />
@@ -154,5 +167,5 @@
         <limit lower="-${PI/2}" upper="${PI/2}" effort="${effort}" velocity="${velocity}" />
     </joint>
-    <joint name="forward_drive_arm_horizontal_arm_joint_3" type="revolute">
+    <joint name="joint_3" type="revolute">
         <parent link="forward_drive_arm_link" />
         <child link="horizontal_arm_link" />
@@ -161,10 +174,10 @@
         <limit lower="-${PI/2}" upper="${PI/2}" effort="${effort}" velocity="${velocity}" />
     </joint>
-    <joint name="horizontal_arm_claw_support_joint" type="fixed">
+    <joint name="horizontal_arm_claw_support" type="fixed">
         <parent link="horizontal_arm_link" />
         <child link="claw_support_link" />
         <origin xyz="0 0.82 0" rpy="0 0 0" />
     </joint>
-    <joint name="claw_support_gripper_right_joint_4" type="revolute">
+    <joint name="joint_4" type="revolute">
         <parent link="claw_support_link" />
         <child link="gripper_right_link" />
@@ -173,5 +186,5 @@
         <limit lower="-${PI/2}" upper="0.0" effort="${effort}" velocity="${velocity}" />
     </joint>
-    <joint name="claw_support_gripper_left_joint_5" type="revolute">
+    <joint name="joint_5" type="revolute">
         <parent link="claw_support_link" />
         <child link="gripper_left_link" />
@@ -181,3 +194,8 @@
         <mimic joint="claw_support_gripper_right_joint_4" multiplier="-1" offset="0" />
     </joint>
+    <!-- transmissions -->
+    <xacro:default_transmission number="1" />
+    <xacro:default_transmission number="2" />
+    <xacro:default_transmission number="3" />
+    <xacro:default_transmission number="4" />
 </robot>

Commit message: fix joint names

File: arduinobot_description/urdf/arduinobot.urdf.xacro (robot description, xacro)
@@ -192,5 +192,5 @@
         <axis xyz="0 0 1" />
         <limit lower="0.0" upper="${PI/2}" effort="${effort}" velocity="${velocity}" />
-        <mimic joint="claw_support_gripper_right_joint_4" multiplier="-1" offset="0" />
+        <mimic joint="joint_4" multiplier="-1" offset="0" />
     </joint>
     <!-- transmissions -->

Commit message: debugging

File: arduinobot_description/urdf/arduinobot.urdf.xacro (robot description, xacro)
@@ -194,4 +194,9 @@
         <mimic joint="joint_4" multiplier="-1" offset="0" />
     </joint>
+    <!-- <link name="dummy_mimic_fix"/>
+    <joint name="joint_5_mimic" type="fixed">
+        <parent link="world" />
+        <child link="dummy_mimic_fix" />
+    </joint> -->
     <!-- transmissions -->
     <xacro:default_transmission number="1" />
