Commit message: experiment with mass

File: arduinobot_description/urdf/arduinobot.urdf.xacro (robot description, xacro)
@@ -13,6 +13,6 @@
             <mass value="${mass}" />
             <inertia ixx="1.0" ixy="0.0" ixz="0.0"
-                iyy="1.0" iyz="0.0"
-                izz="1.0" />
+                     iyy="1.0" iyz="0.0"
+                     izz="1.0" />
         </inertial>
     </xacro:macro>
@@ -29,107 +29,107 @@
     <link name="world" />
     <link name="base_link">
+        <xacro:default_inertial mass="10.0" />
+        <visual>
+            <origin xyz="-0.5 -0.5 0" rpy="0 0 0" />
+            <geometry>
+                <mesh filename="package://arduinobot_description/meshes/basement.STL"
+                    scale="0.01 0.01 0.01" />
+            </geometry>
+        </visual>
+        <collision>
+            <origin xyz="-0.5 -0.5 0" rpy="0 0 0" />
+            <geometry>
+                <mesh filename="package://arduinobot_description/meshes/basement.STL"
+                    scale="0.01 0.01 0.01" />
+            </geometry>
+        </collision>
+    </link>
+    <link name="base_plate_link">
         <xacro:default_inertial mass="1.0" />
         <visual>
-            <origin xyz="-0.5 -0.5 0" rpy="0 0 0" />
-            <geometry>
-                <mesh filename="package://arduinobot_description/meshes/basement.STL"
-                    scale="0.01 0.01 0.01" />
-            </geometry>
-        </visual>
-        <collision>
-            <origin xyz="-0.5 -0.5 0" rpy="0 0 0" />
-            <geometry>
-                <mesh filename="package://arduinobot_description/meshes/basement.STL"
-                    scale="0.01 0.01 0.01" />
-            </geometry>
-        </collision>
-    </link>
-    <link name="base_plate_link">
+            <origin xyz="-0.39 -0.39 -0.56" rpy="0 0 0" />
+            <geometry>
+                <mesh filename="package://arduinobot_description/meshes/base_plate.STL"
+                    scale="0.01 0.01 0.01" />
+            </geometry>
+        </visual>
+        <collision>
+            <origin xyz="-0.39 -0.39 -0.56" rpy="0 0 0" />
+            <geometry>
+                <mesh filename="package://arduinobot_description/meshes/base_plate.STL"
+                    scale="0.01 0.01 0.01" />
+            </geometry>
+        </collision>
+    </link>
+    <link name="forward_drive_arm_link">
+        <xacro:default_inertial mass="1.0" />
+        <visual>
+            <origin xyz="0.19 0.06 -0.08" rpy="0 -${PI/2} ${PI/2}" />
+            <geometry>
+                <mesh filename="package://arduinobot_description/meshes/forward_drive_arm.STL"
+                    scale="0.01 0.01 0.01" />
+            </geometry>
+        </visual>
+        <collision>
+            <origin xyz="0.19 0.06 -0.08" rpy="0 -${PI/2} ${PI/2}" />
+            <geometry>
+                <mesh filename="package://arduinobot_description/meshes/forward_drive_arm.STL"
+                    scale="0.01 0.01 0.01" />
+            </geometry>
+        </collision>
+    </link>
+    <link name="horizontal_arm_link">
+        <xacro:default_inertial mass="1.0" />
+        <visual>
+            <origin xyz="-0.03 -0.4 -0.06" rpy="${PI/2} 0 ${PI/2}" />
+            <geometry>
+                <mesh filename="package://arduinobot_description/meshes/horizontal_arm.STL"
+                    scale="0.01 0.01 0.01" />
+            </geometry>
+        </visual>
+        <collision>
+            <origin xyz="-0.03 -0.4 -0.06" rpy="${PI/2} 0 ${PI/2}" />
+            <geometry>
+                <mesh filename="package://arduinobot_description/meshes/horizontal_arm.STL"
+                    scale="0.01 0.01 0.01" />
+            </geometry>
+        </collision>
+    </link>
+    <link name="claw_support_link">
+        <xacro:default_inertial mass="0.5" />
+        <visual>
+            <origin xyz="0 -0.05 -0.15" rpy="0 0 ${PI/2}" />
+            <geometry>
+                <mesh filename="package://arduinobot_description/meshes/claw_support.STL"
+                    scale="0.01 0.01 0.01" />
+            </geometry>
+        </visual>
+        <collision>
+            <origin xyz="0 -0.05 -0.15" rpy="0 0 ${PI/2}" />
+            <geometry>
+                <mesh filename="package://arduinobot_description/meshes/claw_support.STL"
+                    scale="0.01 0.01 0.01" />
+            </geometry>
+        </collision>
+    </link>
+    <link name="gripper_right_link">
         <xacro:default_inertial mass="0.1" />
         <visual>
-            <origin xyz="-0.39 -0.39 -0.56" rpy="0 0 0" />
-            <geometry>
-                <mesh filename="package://arduinobot_description/meshes/base_plate.STL"
-                    scale="0.01 0.01 0.01" />
-            </geometry>
-        </visual>
-        <collision>
-            <origin xyz="-0.39 -0.39 -0.56" rpy="0 0 0" />
-            <geometry>
-                <mesh filename="package://arduinobot_description/meshes/base_plate.STL"
-                    scale="0.01 0.01 0.01" />
-            </geometry>
-        </collision>
-    </link>
-    <link name="forward_drive_arm_link">
+            <origin xyz="-0.1 0.5 -0.1" rpy="0 0 -${PI/2}" />
+            <geometry>
+                <mesh filename="package://arduinobot_description/meshes/right_finger.STL"
+                    scale="0.01 0.01 0.01" />
+            </geometry>
+        </visual>
+        <collision>
+            <origin xyz="-0.1 0.5 -0.1" rpy="0 0 -${PI/2}" />
+            <geometry>
+                <mesh filename="package://arduinobot_description/meshes/right_finger.STL"
+                    scale="0.01 0.01 0.01" />
+            </geometry>
+        </collision>
+    </link>
+    <link name="gripper_left_link">
         <xacro:default_inertial mass="0.1" />
-        <visual>
-            <origin xyz="0.19 0.06 -0.08" rpy="0 -${PI/2} ${PI/2}" />
-            <geometry>
-                <mesh filename="package://arduinobot_description/meshes/forward_drive_arm.STL"
-                    scale="0.01 0.01 0.01" />
-            </geometry>
-        </visual>
-        <collision>
-            <origin xyz="0.19 0.06 -0.08" rpy="0 -${PI/2} ${PI/2}" />
-            <geometry>
-                <mesh filename="package://arduinobot_description/meshes/forward_drive_arm.STL"
-                    scale="0.01 0.01 0.01" />
-            </geometry>
-        </collision>
-    </link>
-    <link name="horizontal_arm_link">
-        <xacro:default_inertial mass="0.1" />
-        <visual>
-            <origin xyz="-0.03 -0.4 -0.06" rpy="${PI/2} 0 ${PI/2}" />
-            <geometry>
-                <mesh filename="package://arduinobot_description/meshes/horizontal_arm.STL"
-                    scale="0.01 0.01 0.01" />
-            </geometry>
-        </visual>
-        <collision>
-            <origin xyz="-0.03 -0.4 -0.06" rpy="${PI/2} 0 ${PI/2}" />
-            <geometry>
-                <mesh filename="package://arduinobot_description/meshes/horizontal_arm.STL"
-                    scale="0.01 0.01 0.01" />
-            </geometry>
-        </collision>
-    </link>
-    <link name="claw_support_link">
-        <xacro:default_inertial mass="0.05" />
-        <visual>
-            <origin xyz="0 -0.05 -0.15" rpy="0 0 ${PI/2}" />
-            <geometry>
-                <mesh filename="package://arduinobot_description/meshes/claw_support.STL"
-                    scale="0.01 0.01 0.01" />
-            </geometry>
-        </visual>
-        <collision>
-            <origin xyz="0 -0.05 -0.15" rpy="0 0 ${PI/2}" />
-            <geometry>
-                <mesh filename="package://arduinobot_description/meshes/claw_support.STL"
-                    scale="0.01 0.01 0.01" />
-            </geometry>
-        </collision>
-    </link>
-    <link name="gripper_right_link">
-        <xacro:default_inertial mass="0.01" />
-        <visual>
-            <origin xyz="-0.1 0.5 -0.1" rpy="0 0 -${PI/2}" />
-            <geometry>
-                <mesh filename="package://arduinobot_description/meshes/right_finger.STL"
-                    scale="0.01 0.01 0.01" />
-            </geometry>
-        </visual>
-        <collision>
-            <origin xyz="-0.1 0.5 -0.1" rpy="0 0 -${PI/2}" />
-            <geometry>
-                <mesh filename="package://arduinobot_description/meshes/right_finger.STL"
-                    scale="0.01 0.01 0.01" />
-            </geometry>
-        </collision>
-    </link>
-    <link name="gripper_left_link">
-        <xacro:default_inertial mass="0.01" />
         <visual>
             <origin xyz="-0.04 0.5 -0.1" rpy="0 0 -${PI/2}" />

Commit message: Added small changes to get everything working

File: arduinobot_description/urdf/arduinobot.urdf.xacro (robot description, xacro)
@@ -194,9 +194,9 @@
         <mimic joint="joint_4" multiplier="-1" offset="0" />
     </joint>
-    <!-- <link name="dummy_mimic_fix"/>
+    <link name="dummy_mimic_fix"/>
     <joint name="joint_5_mimic" type="fixed">
         <parent link="world" />
         <child link="dummy_mimic_fix" />
-    </joint> -->
+    </joint>
     <!-- transmissions -->
     <xacro:default_transmission number="1" />
